Commit message: 修改控制程序

File: urdf/dog.xacro (robot description, xacro)
@@ -5,5 +5,5 @@
     xmlns:sensor="http://playerstage.sourceforge.net/gazebo/xmlschema/#sensor"
     xmlns:xacro="http://ros.org/wiki/xacro">
-    <link name="map">
+    <link name="body">
         <visual>
             <origin xyz="0.5 1 1.6" rpy="0 0 0" />
@@ -27,5 +27,5 @@
             <origin xyz="${xyz}" rpy="${rpy}" />
             <axis xyz="0 1 0" />
-            <parent link="map"/>
+            <parent link="body"/>
             <child link="up_${linkName}"/>
             <limit effort="3000.0" lower="0.0" upper="1500.548" velocity="0.1"/>

Commit message: 解决了由于肢体放置位置导致的质量分布不均匀身体前倾问题

File: urdf/dog.xacro (robot description, xacro)
@@ -12,5 +12,5 @@
     <link name="body">
         <visual>
-            <origin xyz="0.5 1 1.6" rpy="0 0 0" />
+            <origin xyz="0 0 1.6" rpy="0 0 0" />
             <geometry>
                 <box size="1.2  2  0.2" />
@@ -18,5 +18,5 @@
         </visual>
         <collision name="front_omnileg">
-            <origin xyz="0.5 1 1.6" rpy="0 0 0" />
+            <origin xyz="0 0 1.6" rpy="0 0 0" />
             <geometry>
                 <box size="1.2  2  0.2" />
@@ -114,8 +114,8 @@
         </transmission>
     </xacro:macro>
-    <xacro:leg linkName="leftup" xyz="0 2 1.5" rpy ="0 0 1.57"/>
-    <xacro:leg linkName="leftdown" xyz="0 0 1.5" rpy ="0 0 1.57"/>
-    <xacro:leg linkName="rightup" xyz="1 2 1.5" rpy ="0 0 1.57"/>
-    <xacro:leg linkName="rightdown" xyz="1 0 1.5" rpy ="0 0 1.57"/>
+    <xacro:leg linkName="leftup" xyz="-0.5 1 1.5" rpy ="0 0 1.57"/>
+    <xacro:leg linkName="leftdown" xyz="-0.5 -1 1.5" rpy ="0 0 1.57"/>
+    <xacro:leg linkName="rightup" xyz="0.5 1 1.5" rpy ="0 0 1.57"/>
+    <xacro:leg linkName="rightdown" xyz="0.5 -1 1.5" rpy ="0 0 1.57"/>
     <gazebo>
         <plugin name="gazebo_ros_control" filename="libgazebo_ros_control.so">

Commit message: 改进控制

File: urdf/dog.xacro (robot description, xacro)
@@ -24,5 +24,5 @@
         </collision>
         <inertial>
-            <mass value="6.0"/>
+            <mass value="8.0"/>
             <inertia ixx="0.4" ixy="0.0" ixz="0.0" iyy="0.4" iyz="0.0" izz="0.2"/>
         </inertial>
@@ -54,5 +54,5 @@
             </collision>
             <inertial>
-                <mass value="1.0"/>
+                <mass value="0.4"/>
                 <inertia ixx="0.4" ixy="0.0" ixz="0.0" iyy="0.4" iyz="0.0" izz="0.2"/>
             </inertial>
@@ -83,5 +83,5 @@
             </collision>
             <inertial>
-                <mass value="2.0"/>
+                <mass value="0.4"/>
                 <inertia ixx="0.4" ixy="0.0" ixz="0.0" iyy="0.4" iyz="0.0" izz="0.2"/>
             </inertial>
