Commit message: 修改机器狗的参数，并且支持在gazebo中显示

File: urdf/car.xacro (robot description, xacro)
@@ -142,5 +142,5 @@
         <hardwareInterface>hardware_interface/VelocityJointInterface</hardwareInterface>
       </joint>
-      <actuator name="motor_${linkName}">
+      <actuator name="motor_base_to__${linkName}">
         <hardwareInterface>hardware_interface/VelocityJointInterface</hardwareInterface>
         <mechanicalReduction>1</mechanicalReduction>

File: urdf/dog.xacro (robot description, xacro)
@@ -1,4 +1,5 @@
 <?xml version="1.0"?>
-<robot name="cartest" xmlns:controller="http://playerstage.sourceforge.net/gazebo/xmlschema/#controller"
+<robot name="cartest"
+  xmlns:controller="http://playerstage.sourceforge.net/gazebo/xmlschema/#controller"
   xmlns:interface="http://playerstage.sourceforge.net/gazebo/xmlschema/#interface"
   xmlns:sensor="http://playerstage.sourceforge.net/gazebo/xmlschema/#sensor"
@@ -6,84 +7,111 @@
   <link name="map">
     <visual>
-    <origin xyz="0.5 1 1.6" rpy="0 0 0" />
+      <origin xyz="0.5 1 1.6" rpy="0 0 0" />
       <geometry>
-        <box  size="1  2  0.2" />
+        <box size="1.2  2  0.2" />
       </geometry>
     </visual>`
-    <collision name="front_omniwheel">
-      <origin xyz="0.5 1 1" rpy="0 0 0" />
+    <collision name="front_omnileg">
+      <origin xyz="0.5 1 1.6" rpy="0 0 0" />
       <geometry>
-        <box  size="1  2  0.2" />
+        <box size="1.2  2  0.2" />
       </geometry>
     </collision>
     <inertial>
-      <mass value="10.0"/>>
-      <inertia ixx="0.4" ixy="0.0" ixz="0.0" iyy="0.4" iyz="0.0" izz="0.2"/>>
+      <mass value="10.0"/>
+      <inertia ixx="0.4" ixy="0.0" ixz="0.0" iyy="0.4" iyz="0.0" izz="0.2"/>
     </inertial>
   </link>
-<xacro:macro name="wheel" params="linkName xyz rpy">
-<joint name="base_to_${linkName}" type="continuous">
-   <origin xyz="${xyz}" rpy="${rpy}" />
-   <axis xyz="0 1 0" />
-    <parent link="map"/>
-    <child link="up_${linkName}"/>
-  </joint>
+  <xacro:macro name="leg" params="linkName xyz rpy">
+    <joint name="base_to_${linkName}" type="continuous">
+      <origin xyz="${xyz}" rpy="${rpy}" />
+      <axis xyz="0 1 0" />
+      <parent link="map"/>
+      <child link="up_${linkName}"/>
+      <limit effort="1000000.0" lower="0.0" upper="10000.548" velocity="5000"/>
+    </joint>
     <link name="up_${linkName}">
       <visual>
-       <origin xyz="0 0 -0.45" rpy="0 0.4 0" />
+        <origin xyz="0 0 -0.35" rpy="0 0 0" />
         <geometry>
-          <cylinder length="1" radius="0.05"/>
+          <cylinder length="0.7" radius="0.05"/>
         </geometry>
         <material name = "white">
           <color rgba = "0 0 1 1"/>
-      </material>
-    </visual>
-    <collision name="collision_${linkName}">
-   <origin xyz="0 0 -0.45" rpy="0 0.4 0" />
+        </material>
+      </visual>
+      <collision name="collision_${linkName}">
+        <origin xyz="0 0 -0.35" rpy="0 0 0" />
         <geometry>
-          <cylinder length="1" radius="0.05"/>
+          <cylinder length="0.7" radius="0.05"/>
         </geometry>
-    </collision>
-    <inertial>
-      <mass value="2.0"/>>
-      <inertia ixx="0.4" ixy="0.0" ixz="0.0" iyy="0.4" iyz="0.0" izz="0.2"/>>
-    </inertial>
-  </link>
-  <joint name="joint_${linkName}" type="continuous">
-   <origin xyz="0 0 -0.9" rpy="0 0 0" />
-   <axis xyz="0 1 0" />
-    <parent link="up_${linkName}"/>
-    <child link="down_${linkName}"/>
-  </joint>
-<link name="down_${linkName}">
+      </collision>
+      <inertial>
+        <mass value="2.0"/>
+        <inertia ixx="0.4" ixy="0.0" ixz="0.0" iyy="0.4" iyz="0.0" izz="0.2"/>
+      </inertial>
+    </link>
+    <joint name="joint_${linkName}" type="continuous">
+      <origin xyz="0 0 -0.7" rpy="0 0 0" />
+      <axis xyz="0 1 0" />
+      <parent link="up_${linkName}"/>
+      <child link="down_${linkName}"/>
+    </joint>
+    <link name="down_${linkName}">
       <visual>
-       <origin xyz="0 0 -0.45" rpy="0 2.74 0" />
+        <origin xyz="0 0 -0.35" rpy="0 0 0" />
         <geometry>
-          <cylinder length="1" radius="0.05"/>
+          <cylinder length="0.7" radius="0.05"/>
         </geometry>
         <material name = "white">
           <color rgba = "0 0 1 1"/>
-      </material>
-    </visual>
-    <collision name="collision_${linkName}">
-    <origin xyz="0 0 -0.45" rpy="0 2.74 0" />
+        </material>
+      </visual>
+      <collision name="collision_${linkName}">
+        <origin xyz="0 0 -0.35" rpy="0 0 0" />
         <geometry>
-          <cylinder length="1" radius="0.05"/>
+          <cylinder length="0.7" radius="0.05"/>
         </geometry>
-    </collision>
-    <inertial>
-      <mass value="2.0"/>>
-      <inertia ixx="0.4" ixy="0.0" ixz="0.0" iyy="0.4" iyz="0.0" izz="0.2"/>>
-    </inertial>
-  </link>
-</xacro:macro>
-<xacro:wheel linkName="leftup" xyz="0 2 1.5" rpy ="0 0 1.57"/>
-<xacro:wheel linkName="leftdown" xyz="0 0 1.5" rpy ="0 0 1.57"/>
-<xacro:wheel linkName="rightup" xyz="1 2 1.5" rpy ="0 0 1.57"/>
-<xacro:wheel linkName="rightdown" xyz="1 0 1.5" rpy ="0 0 1.57"/>
-<gazebo>
+      </collision>
+      <inertial>
+        <mass value="2.0"/>
+        <inertia ixx="0.4" ixy="0.0" ixz="0.0" iyy="0.4" iyz="0.0" izz="0.2"/>
+      </inertial>
+    </link>
+    <gazebo reference="up_${linkName}">
+      <material>Gazebo/blue</material>
+    </gazebo>
+    <gazebo reference="down_${linkName}">
+      <material>Gazebo/blue</material>
+    </gazebo>
+    <transmission name="tran${linkName}">
+      <type>transmission_interface/SimpleTransmission</type>
+      <joint name="base_to_${linkName}">
+        <hardwareInterface>hardware_interface/VelocityJointInterface</hardwareInterface>
+      </joint>
+      <actuator name="joint_${linkName}">
+        <hardwareInterface>hardware_interface/VelocityJointInterface</hardwareInterface>
+        <mechanicalReduction>1</mechanicalReduction>
+      </actuator>
+    </transmission>
+  <transmission name="tran${linkName}">
+      <type>transmission_interface/SimpleTransmission</type>
+      <joint name="joint_${linkName}">
+        <hardwareInterface>hardware_interface/VelocityJointInterface</hardwareInterface>
+      </joint>
+      <actuator name="motor_joint_${linkName}">
+        <hardwareInterface>hardware_interface/VelocityJointInterface</hardwareInterface>
+        <mechanicalReduction>1</mechanicalReduction>
+      </actuator>
+    </transmission>
+  </xacro:macro>
+  <xacro:leg linkName="leftup" xyz="0 2 1.5" rpy ="0 0 1.57"/>
+  <xacro:leg linkName="leftdown" xyz="0 0 1.5" rpy ="0 0 1.57"/>
+  <xacro:leg linkName="rightup" xyz="1 2 1.5" rpy ="0 0 1.57"/>
+  <xacro:leg linkName="rightdown" xyz="1 0 1.5" rpy ="0 0 1.57"/>
+  <gazebo>
     <plugin name="gazebo_ros_control" filename="libgazebo_ros_control.so">
       <robotNamespace>/</robotNamespace>
     </plugin>
-</gazebo>
+  </gazebo>
 </robot>

Commit message: 提交

File: urdf/car.xacro (robot description, xacro)
@@ -21,7 +21,5 @@
       <origin xyz="0.5 1 1.1" rpy="0 0 0" />
       <mass value="1.0"/>
->
       <inertia ixx="0.4" ixy="0.0" ixz="0.0" iyy="0.4" iyz="0.0" izz="0.2"/>
->
     </inertial>
   </link>

File: urdf/dog.xacro (robot description, xacro)
@@ -1,117 +1,120 @@
 <?xml version="1.0"?>
 <robot name="cartest"
-  xmlns:controller="http://playerstage.sourceforge.net/gazebo/xmlschema/#controller"
-  xmlns:interface="http://playerstage.sourceforge.net/gazebo/xmlschema/#interface"
-  xmlns:sensor="http://playerstage.sourceforge.net/gazebo/xmlschema/#sensor"
-  xmlns:xacro="http://ros.org/wiki/xacro">
-  <link name="map">
-    <visual>
-      <origin xyz="0.5 1 1.6" rpy="0 0 0" />
-      <geometry>
-        <box size="1.2  2  0.2" />
-      </geometry>
-    </visual>`
-    <collision name="front_omnileg">
-      <origin xyz="0.5 1 1.6" rpy="0 0 0" />
-      <geometry>
-        <box size="1.2  2  0.2" />
-      </geometry>
-    </collision>
-    <inertial>
-      <mass value="10.0"/>
-      <inertia ixx="0.4" ixy="0.0" ixz="0.0" iyy="0.4" iyz="0.0" izz="0.2"/>
-    </inertial>
-  </link>
-  <xacro:macro name="leg" params="linkName xyz rpy">
-    <joint name="base_to_${linkName}" type="continuous">
-      <origin xyz="${xyz}" rpy="${rpy}" />
-      <axis xyz="0 1 0" />
-      <parent link="map"/>
-      <child link="up_${linkName}"/>
-      <limit effort="1000000.0" lower="0.0" upper="10000.548" velocity="5000"/>
-    </joint>
-    <link name="up_${linkName}">
-      <visual>
-        <origin xyz="0 0 -0.35" rpy="0 0 0" />
-        <geometry>
-          <cylinder length="0.7" radius="0.05"/>
-        </geometry>
-        <material name = "white">
-          <color rgba = "0 0 1 1"/>
-        </material>
-      </visual>
-      <collision name="collision_${linkName}">
-        <origin xyz="0 0 -0.35" rpy="0 0 0" />
-        <geometry>
-          <cylinder length="0.7" radius="0.05"/>
-        </geometry>
-      </collision>
-      <inertial>
-        <mass value="2.0"/>
-        <inertia ixx="0.4" ixy="0.0" ixz="0.0" iyy="0.4" iyz="0.0" izz="0.2"/>
-      </inertial>
+    xmlns:controller="http://playerstage.sourceforge.net/gazebo/xmlschema/#controller"
+    xmlns:interface="http://playerstage.sourceforge.net/gazebo/xmlschema/#interface"
+    xmlns:sensor="http://playerstage.sourceforge.net/gazebo/xmlschema/#sensor"
+    xmlns:xacro="http://ros.org/wiki/xacro">
+    <link name="map">
+        <visual>
+            <origin xyz="0.5 1 1.6" rpy="0 0 0" />
+            <geometry>
+                <box size="1.2  2  0.2" />
+            </geometry>
+        </visual>
+        <collision name="front_omnileg">
+            <origin xyz="0.5 1 1.6" rpy="0 0 0" />
+            <geometry>
+                <box size="1.2  2  0.2" />
+            </geometry>
+        </collision>
+        <inertial>
+            <mass value="2.0"/>
+            <inertia ixx="0.4" ixy="0.0" ixz="0.0" iyy="0.4" iyz="0.0" izz="0.2"/>
+        </inertial>
     </link>
-    <joint name="joint_${linkName}" type="continuous">
-      <origin xyz="0 0 -0.7" rpy="0 0 0" />
-      <axis xyz="0 1 0" />
-      <parent link="up_${linkName}"/>
-      <child link="down_${linkName}"/>
-    </joint>
-    <link name="down_${linkName}">
-      <visual>
-        <origin xyz="0 0 -0.35" rpy="0 0 0" />
-        <geometry>
-          <cylinder length="0.7" radius="0.05"/>
-        </geometry>
-        <material name = "white">
-          <color rgba = "0 0 1 1"/>
-        </material>
-      </visual>
-      <collision name="collision_${linkName}">
-        <origin xyz="0 0 -0.35" rpy="0 0 0" />
-        <geometry>
-          <cylinder length="0.7" radius="0.05"/>
-        </geometry>
-      </collision>
-      <inertial>
-        <mass value="2.0"/>
-        <inertia ixx="0.4" ixy="0.0" ixz="0.0" iyy="0.4" iyz="0.0" izz="0.2"/>
-      </inertial>
-    </link>
-    <gazebo reference="up_${linkName}">
-      <material>Gazebo/blue</material>
+    <xacro:macro name="leg" params="linkName xyz rpy">
+        <joint name="base_to_${linkName}" type="continuous">
+            <origin xyz="${xyz}" rpy="${rpy}" />
+            <axis xyz="0 1 0" />
+            <parent link="map"/>
+            <child link="up_${linkName}"/>
+            <limit effort="3000.0" lower="0.0" upper="1500.548" velocity="0.1"/>
+            <dynamics damping="0.2"/>
+        </joint>
+        <link name="up_${linkName}">
+            <visual>
+                <origin xyz="0 0 -0.35" rpy="0 0 0" />
+                <geometry>
+                    <cylinder length="0.7" radius="0.05"/>
+                </geometry>
+                <material name = "white">
+                    <color rgba = "0 0 1 1"/>
+                </material>
+            </visual>
+            <collision name="collision_${linkName}">
+                <origin xyz="0 0 -0.35" rpy="0 0 0" />
+                <geometry>
+                    <cylinder length="0.7" radius="0.05"/>
+                </geometry>
+            </collision>
+            <inertial>
+                <mass value="1.0"/>
+                <inertia ixx="0.4" ixy="0.0" ixz="0.0" iyy="0.4" iyz="0.0" izz="0.2"/>
+            </inertial>
+        </link>
+        <joint name="joint_${linkName}" type="continuous">
+            <origin xyz="0 0 -0.7" rpy="0 0 0" />
+            <axis xyz="0 1 0" />
+            <parent link="up_${linkName}"/>
+            <child link="down_${linkName}"/>
+            <limit effort="3000.0" lower="0.0" upper="1500.548" velocity="0.1"/>
+            <dynamics damping="0.2"/>
+        </joint>
+        <link name="down_${linkName}">
+            <visual>
+                <origin xyz="0 0 -0.35" rpy="0 0 0" />
+                <geometry>
+                    <cylinder length="0.7" radius="0.05"/>
+                </geometry>
+                <material name = "white">
+                    <color rgba = "0 0 1 1"/>
+                </material>
+            </visual>
+            <collision name="collision_${linkName}">
+                <origin xyz="0 0 -0.35" rpy="0 0 0" />
+                <geometry>
+                    <cylinder length="0.7" radius="0.05"/>
+                </geometry>
+            </collision>
+            <inertial>
+                <mass value="1.0"/>
+                <inertia ixx="0.4" ixy="0.0" ixz="0.0" iyy="0.4" iyz="0.0" izz="0.2"/>
+            </inertial>
+        </link>
+        <gazebo reference="up_${linkName}">
+            <material>Gazebo/blue</material>
+        </gazebo>
+        <gazebo reference="down_${linkName}">
+            <material>Gazebo/blue</material>
+        </gazebo>
+        <transmission name="tran${linkName}">
+            <type>transmission_interface/SimpleTransmission</type>
+            <joint name="base_to_${linkName}">
+                <hardwareInterface>hardware_interface/EffortJointInterface</hardwareInterface>
+            </joint>
+            <actuator name="joint_${linkName}">
+                <hardwareInterface>hardware_interface/EffortJointInterface</hardwareInterface>
+                <mechanicalReduction>1</mechanicalReduction>
+            </actuator>
+        </transmission>
+        <transmission name="tran${linkName}">
+            <type>transmission_interface/SimpleTransmission</type>
+            <joint name="joint_${linkName}">
+                <hardwareInterface>hardware_interface/EffortJointInterface</hardwareInterface>
+            </joint>
+            <actuator name="motor_joint_${linkName}">
+                <hardwareInterface>hardware_interface/EffortJointInterface</hardwareInterface>
+                <mechanicalReduction>1</mechanicalReduction>
+            </actuator>
+        </transmission>
+    </xacro:macro>
+    <xacro:leg linkName="leftup" xyz="0 2 1.5" rpy ="0 0 1.57"/>
+    <xacro:leg linkName="leftdown" xyz="0 0 1.5" rpy ="0 0 1.57"/>
+    <xacro:leg linkName="rightup" xyz="1 2 1.5" rpy ="0 0 1.57"/>
+    <xacro:leg linkName="rightdown" xyz="1 0 1.5" rpy ="0 0 1.57"/>
+    <gazebo>
+        <plugin name="gazebo_ros_control" filename="libgazebo_ros_control.so">
+            <robotNamespace>/</robotNamespace>
+        </plugin>
     </gazebo>
-    <gazebo reference="down_${linkName}">
-      <material>Gazebo/blue</material>
-    </gazebo>
-    <transmission name="tran${linkName}">
-      <type>transmission_interface/SimpleTransmission</type>
-      <joint name="base_to_${linkName}">
-        <hardwareInterface>hardware_interface/VelocityJointInterface</hardwareInterface>
-      </joint>
-      <actuator name="joint_${linkName}">
-        <hardwareInterface>hardware_interface/VelocityJointInterface</hardwareInterface>
-        <mechanicalReduction>1</mechanicalReduction>
-      </actuator>
-    </transmission>
-  <transmission name="tran${linkName}">
-      <type>transmission_interface/SimpleTransmission</type>
-      <joint name="joint_${linkName}">
-        <hardwareInterface>hardware_interface/VelocityJointInterface</hardwareInterface>
-      </joint>
-      <actuator name="motor_joint_${linkName}">
-        <hardwareInterface>hardware_interface/VelocityJointInterface</hardwareInterface>
-        <mechanicalReduction>1</mechanicalReduction>
-      </actuator>
-    </transmission>
-  </xacro:macro>
-  <xacro:leg linkName="leftup" xyz="0 2 1.5" rpy ="0 0 1.57"/>
-  <xacro:leg linkName="leftdown" xyz="0 0 1.5" rpy ="0 0 1.57"/>
-  <xacro:leg linkName="rightup" xyz="1 2 1.5" rpy ="0 0 1.57"/>
-  <xacro:leg linkName="rightdown" xyz="1 0 1.5" rpy ="0 0 1.57"/>
-  <gazebo>
-    <plugin name="gazebo_ros_control" filename="libgazebo_ros_control.so">
-      <robotNamespace>/</robotNamespace>
-    </plugin>
-  </gazebo>
 </robot>
