Commit message: 同时对四只脚进行控制，但是控制的很差，需要改进

File: urdf/car.xacro (robot description, xacro)
@@ -1,158 +1,143 @@
 <?xml version="1.0"?>
 <robot name="cartest"
-  xmlns:controller="http://playerstage.sourceforge.net/gazebo/xmlschema/#controller"
-  xmlns:interface="http://playerstage.sourceforge.net/gazebo/xmlschema/#interface"
-  xmlns:sensor="http://playerstage.sourceforge.net/gazebo/xmlschema/#sensor"
-  xmlns:xacro="http://ros.org/wiki/xacro">
-  <link name="base_footprint">
-    <visual>
-      <origin xyz="0.5 1 1.1" rpy="0 0 0" />
-      <geometry>
-        <box size="1  2  0.25" />
-      </geometry>
-    </visual>
-    <collision>
-      <origin xyz="0.5 1 1.1" rpy="0 0 0" />
-      <geometry>
-        <box size="1  2  0.25" />
-      </geometry>
-    </collision>
-    <inertial>
-      <origin xyz="0.5 1 1.1" rpy="0 0 0" />
-      <mass value="1.0"/>
-      <inertia ixx="0.4" ixy="0.0" ixz="0.0" iyy="0.4" iyz="0.0" izz="0.2"/>
-    </inertial>
-  </link>
-  <gazebo reference="base_footprint">
-    <material>Gazebo/white</material>
-  </gazebo>
-  <link name="hokuyo_link">
-    <inertial>
-      <origin xyz="0.0 0.0 -0.2" rpy="0.0 0.0 0.0"/>
-      <mass value="0.2"/>
-      <inertia ixx="0.0" ixy="0.0" ixz="0.0" iyy="0.0" iyz="0.0" izz="0.0"/>
-    </inertial>
-    <visual>
-      <origin xyz="0.0 0.0 0.0" rpy="0.0 0.0 0.0"/>
-      <geometry>
-        <box size="0.2 0.2 0.2"/>
-      </geometry>
-      <material >
-        <color rgba="1.0 0.0 0.0 1.0"/>
-      </material>
-    </visual>
-    <collision>
-      <origin xyz="0.0 0.0 0.0" rpy="0.0 0.0 0.0"/>
-      <geometry>
-        <box size="0.2 0.2 0.2"/>
-      </geometry>
-    </collision>
-  </link>
-  <gazebo reference="hokuyo_link">
-    <sensor type="ray" name="head_hokuyo_sensor">
-      <pose>0.3 0.3 0.3 0 0 0</pose>
-      <visualize>true</visualize>
-      <update_rate>10</update_rate>
-      <ray>
-        <scan>
-          <horizontal>
-            <samples>480</samples>
-            <resolution>1</resolution>
-            <min_angle>-3.14</min_angle>
-            <max_angle>3.14</max_angle>
-          </horizontal>
-        </scan>
-        <range>
-          <min>0.10</min>
-          <max>30.0</max>
-          <resolution>0.01</resolution>
-        </range>
-        <noise>
-          <type>gaussian</type>
-          <mean>0.0</mean>
-          <stddev>0.01</stddev>
-        </noise>
-      </ray>
-      <plugin name="gazebo_ros_head_hokuyo_controller" filename="libgazebo_ros_laser.so">
-        <topicName>scan</topicName>
-        <frameName>hokuyo_link</frameName>
-      </plugin>
-    </sensor>
-  </gazebo>
-  <joint name="joint_name" type="fixed">
-    <origin xyz="0.25 0.8 1.7" rpy="0.0 0.0 0.0"/>
-    <parent link="base_footprint"/>
-    <child link="hokuyo_link"/>
-  </joint>
-  <!-- <link name="imu_link"/>
-  <joint name="base_to_imu" type="fixed">
-    <axis rpy="0 0 0" xyz="0 0 0"/>
-    <parent link="base_link"/>
-    <child link="imu_link"/>
-    <origin rpy="0 0 0" xyz="0 0 .2"/>
-  </joint> -->
-  <xacro:macro name="wheel" params="linkName xyz rpy">
-    <joint name="base_to_${linkName}" type="continuous">
-      <origin xyz="${xyz}" rpy="${rpy}" />
-      <axis xyz="1 0 0" />
-      <parent link="base_footprint"/>
-      <child link="${linkName}"/>
-      <limit effort="1000000.0" lower="0.0" upper="10000.548" velocity="5000"/>
+    xmlns:controller="http://playerstage.sourceforge.net/gazebo/xmlschema/#controller"
+    xmlns:interface="http://playerstage.sourceforge.net/gazebo/xmlschema/#interface"
+    xmlns:sensor="http://playerstage.sourceforge.net/gazebo/xmlschema/#sensor"
+    xmlns:xacro="http://ros.org/wiki/xacro">
+    <link name="base_footprint">
+        <visual>
+            <origin xyz="0.5 1 1.1" rpy="0 0 0" />
+            <geometry>
+                <box size="1  2  0.25" />
+            </geometry>
+        </visual>
+        <collision>
+            <origin xyz="0.5 1 1.1" rpy="0 0 0" />
+            <geometry>
+                <box size="1  2  0.25" />
+            </geometry>
+        </collision>
+        <inertial>
+            <origin xyz="0.5 1 1.1" rpy="0 0 0" />
+            <mass value="1.0"/>
+            <inertia ixx="0.4" ixy="0.0" ixz="0.0" iyy="0.4" iyz="0.0" izz="0.2"/>
+        </inertial>
+    </link>
+    <gazebo reference="base_footprint">
+        <material>Gazebo/white</material>
+    </gazebo>
+    <link name="hokuyo_link">
+        <inertial>
+            <origin xyz="0.0 0.0 -0.2" rpy="0.0 0.0 0.0"/>
+            <mass value="0.2"/>
+            <inertia ixx="0.0" ixy="0.0" ixz="0.0" iyy="0.0" iyz="0.0" izz="0.0"/>
+        </inertial>
+        <visual>
+            <origin xyz="0.0 0.0 0.0" rpy="0.0 0.0 0.0"/>
+            <geometry>
+                <box size="0.2 0.2 0.2"/>
+            </geometry>
+            <material >
+                <color rgba="1.0 0.0 0.0 1.0"/>
+            </material>
+        </visual>
+        <collision>
+            <origin xyz="0.0 0.0 0.0" rpy="0.0 0.0 0.0"/>
+            <geometry>
+                <box size="0.2 0.2 0.2"/>
+            </geometry>
+        </collision>
+    </link>
+    <gazebo reference="hokuyo_link">
+        <sensor type="ray" name="head_hokuyo_sensor">
+            <pose>0.3 0.3 0.3 0 0 0</pose>
+            <visualize>true</visualize>
+            <update_rate>10</update_rate>
+            <ray>
+                <scan>
+                    <horizontal>
+                        <samples>480</samples>
+                        <resolution>1</resolution>
+                        <min_angle>-3.14</min_angle>
+                        <max_angle>3.14</max_angle>
+                    </horizontal>
+                </scan>
+                <range>
+                    <min>0.10</min>
+                    <max>30.0</max>
+                    <resolution>0.01</resolution>
+                </range>
+                <noise>
+                    <type>gaussian</type>
+                    <mean>0.0</mean>
+                    <stddev>0.01</stddev>
+                </noise>
+            </ray>
+            <plugin name="gazebo_ros_head_hokuyo_controller" filename="libgazebo_ros_laser.so">
+                <topicName>scan</topicName>
+                <frameName>hokuyo_link</frameName>
+            </plugin>
+        </sensor>
+    </gazebo>
+    <joint name="joint_name" type="fixed">
+        <origin xyz="0.25 0.8 1.7" rpy="0.0 0.0 0.0"/>
+        <parent link="base_footprint"/>
+        <child link="hokuyo_link"/>
     </joint>
-    <link name="${linkName}">
-      <visual>
-        <origin xyz="0 0 0" rpy="0 1.57 0" />
-        <geometry>
-          <cylinder length="0.2" radius="0.35"/>
-        </geometry>
-        <material name = "white">
-          <color rgba = "0 0 1 1"/>
-        </material>
-      </visual>
-      <collision name="collision_${linkName}">
-        <origin xyz="0 0 0" rpy="0 1.57 0" />
-        <geometry>
-          <cylinder length="0.2" radius="0.35"/>
-        </geometry>
-      </collision>
-      <inertial>
-        <origin xyz="0 0 0" rpy="0 1.57 0" />
-        <mass value="1.0"/>
-        <inertia ixx="0.4" ixy="0.0" ixz="0.0" iyy="0.4" iyz="0.0" izz="0.2"/>
-      </inertial>
-    </link>
-    <!-- <transmission name="tran${linkName}">
-    <type>transmission_interface/SimpleTransmission</type>
-    <joint name="base_to_${linkName}">
-      <hardwareInterface>hardware_interface/EffortJointInterface</hardwareInterface>
-    </joint>
-    <actuator name="motor_${linkName}">
-      <hardwareInterface>hardware_interface/EffortJointInterface</hardwareInterface>
-      <mechanicalReduction>1</mechanicalReduction>
-    </actuator>
-  </transmission> -->
-    <gazebo reference="${linkName}">
-      <material>Gazebo/Orange</material>
+    <!-- <link name="imu_link"/><joint name="base_to_imu" type="fixed"><axis rpy="0 0 0" xyz="0 0 0"/><parent link="base_link"/><child link="imu_link"/><origin rpy="0 0 0" xyz="0 0 .2"/></joint> -->
+    <xacro:macro name="wheel" params="linkName xyz rpy">
+        <joint name="base_to_${linkName}" type="continuous">
+            <origin xyz="${xyz}" rpy="${rpy}" />
+            <axis xyz="1 0 0" />
+            <parent link="base_footprint"/>
+            <child link="${linkName}"/>
+            <limit effort="1000000.0" lower="0.0" upper="10000.548" velocity="5000"/>
+        </joint>
+        <link name="${linkName}">
+            <visual>
+                <origin xyz="0 0 0" rpy="0 1.57 0" />
+                <geometry>
+                    <cylinder length="0.2" radius="0.35"/>
+                </geometry>
+                <material name = "white">
+                    <color rgba = "0 0 1 1"/>
+                </material>
+            </visual>
+            <collision name="collision_${linkName}">
+                <origin xyz="0 0 0" rpy="0 1.57 0" />
+                <geometry>
+                    <cylinder length="0.2" radius="0.35"/>
+                </geometry>
+            </collision>
+            <inertial>
+                <origin xyz="0 0 0" rpy="0 1.57 0" />
+                <mass value="1.0"/>
+                <inertia ixx="0.4" ixy="0.0" ixz="0.0" iyy="0.4" iyz="0.0" izz="0.2"/>
+            </inertial>
+        </link>
+        <!-- <transmission name="tran${linkName}"><type>transmission_interface/SimpleTransmission</type><joint name="base_to_${linkName}"><hardwareInterface>hardware_interface/EffortJointInterface</hardwareInterface></joint><actuator name="motor_${linkName}"><hardwareInterface>hardware_interface/EffortJointInterface</hardwareInterface><mechanicalReduction>1</mechanicalReduction></actuator></transmission> -->
+        <gazebo reference="${linkName}">
+            <material>Gazebo/Orange</material>
+        </gazebo>
+        <transmission name="tran${linkName}">
+            <type>transmission_interface/SimpleTransmission</type>
+            <joint name="base_to_${linkName}">
+                <hardwareInterface>hardware_interface/VelocityJointInterface</hardwareInterface>
+            </joint>
+            <actuator name="motor_base_to__${linkName}">
+                <hardwareInterface>hardware_interface/VelocityJointInterface</hardwareInterface>
+                <mechanicalReduction>1</mechanicalReduction>
+            </actuator>
+        </transmission>
+    </xacro:macro>
+    <xacro:wheel linkName="leftup" xyz="0 2 0.5" rpy ="0 0 0"/>
+    <xacro:wheel linkName="leftdown" xyz="0 0 0.5" rpy ="0 0 0"/>
+    <xacro:wheel linkName="rightup" xyz="1 2 0.5" rpy ="0 0 0"/>
+    <xacro:wheel linkName="rightdown" xyz="1 0 0.5" rpy ="0 0 0"/>
+    <gazebo>
+        <plugin name="gazebo_ros_control" filename="libgazebo_ros_control.so">
+            <robotNamespace>/</robotNamespace>
+            <robotSimType>gazebo_ros_control/DefaultRobotHWSim</robotSimType>
+        </plugin>
     </gazebo>
-    <transmission name="tran${linkName}">
-      <type>transmission_interface/SimpleTransmission</type>
-      <joint name="base_to_${linkName}">
-        <hardwareInterface>hardware_interface/VelocityJointInterface</hardwareInterface>
-      </joint>
-      <actuator name="motor_base_to__${linkName}">
-        <hardwareInterface>hardware_interface/VelocityJointInterface</hardwareInterface>
-        <mechanicalReduction>1</mechanicalReduction>
-      </actuator>
-    </transmission>
-  </xacro:macro>
-  <xacro:wheel linkName="leftup" xyz="0 2 0.5" rpy ="0 0 0"/>
-  <xacro:wheel linkName="leftdown" xyz="0 0 0.5" rpy ="0 0 0"/>
-  <xacro:wheel linkName="rightup" xyz="1 2 0.5" rpy ="0 0 0"/>
-  <xacro:wheel linkName="rightdown" xyz="1 0 0.5" rpy ="0 0 0"/>
-  <gazebo>
-    <plugin name="gazebo_ros_control" filename="libgazebo_ros_control.so">
-      <robotNamespace>/</robotNamespace>
-      <robotSimType>gazebo_ros_control/DefaultRobotHWSim</robotSimType>
-    </plugin>
-  </gazebo>
 </robot>

File: urdf/dog.xacro (robot description, xacro)
@@ -5,4 +5,9 @@
     xmlns:sensor="http://playerstage.sourceforge.net/gazebo/xmlschema/#sensor"
     xmlns:xacro="http://ros.org/wiki/xacro">
+    <!--<link name="world"/>
+    <joint name="test" type="fixed">
+        <parent link="world"/>
+        <child link="body"/>
+    </joint>-->
     <link name="body">
         <visual>
@@ -29,5 +34,5 @@
             <parent link="body"/>
             <child link="up_${linkName}"/>
-            <limit effort="3000.0" lower="0.0" upper="1500.548" velocity="0.1"/>
+            <limit effort="3000.0" lower="0.0" upper="3000.548" velocity="0.2"/>
             <dynamics damping="0.2"/>
         </joint>
@@ -58,5 +63,5 @@
             <parent link="up_${linkName}"/>
             <child link="down_${linkName}"/>
-            <limit effort="3000.0" lower="0.0" upper="1500.548" velocity="0.1"/>
+            <limit effort="3000.0" lower="0.0" upper="3000.548" velocity="0.2"/>
             <dynamics damping="0.2"/>
         </joint>

Commit message: 增加人形模型

File: urdf/car.xacro (robot description, xacro)
@@ -19,5 +19,4 @@
         </collision>
         <inertial>
-            <origin xyz="0.5 1 1.1" rpy="0 0 0" />
             <mass value="1.0"/>
             <inertia ixx="0.4" ixy="0.0" ixz="0.0" iyy="0.4" iyz="0.0" izz="0.2"/>

File: urdf/dog.xacro (robot description, xacro)
@@ -24,5 +24,5 @@
         </collision>
         <inertial>
-            <mass value="2.0"/>
+            <mass value="6.0"/>
             <inertia ixx="0.4" ixy="0.0" ixz="0.0" iyy="0.4" iyz="0.0" izz="0.2"/>
         </inertial>
@@ -34,5 +34,5 @@
             <parent link="body"/>
             <child link="up_${linkName}"/>
-            <limit effort="3000.0" lower="0.0" upper="3000.548" velocity="0.2"/>
+            <limit effort="2000.0" lower="0.0" upper="2000.548" velocity="0.7"/>
             <dynamics damping="0.2"/>
         </joint>
@@ -63,5 +63,5 @@
             <parent link="up_${linkName}"/>
             <child link="down_${linkName}"/>
-            <limit effort="3000.0" lower="0.0" upper="3000.548" velocity="0.2"/>
+            <limit effort="2000.0" lower="0.0" upper="2000.548" velocity="0.7"/>
             <dynamics damping="0.2"/>
         </joint>
@@ -83,5 +83,5 @@
             </collision>
             <inertial>
-                <mass value="1.0"/>
+                <mass value="2.0"/>
                 <inertia ixx="0.4" ixy="0.0" ixz="0.0" iyy="0.4" iyz="0.0" izz="0.2"/>
             </inertial>
@@ -96,8 +96,8 @@
             <type>transmission_interface/SimpleTransmission</type>
             <joint name="base_to_${linkName}">
-                <hardwareInterface>hardware_interface/EffortJointInterface</hardwareInterface>
+                <hardwareInterface>hardware_interface/VelocityJointInterface</hardwareInterface>
             </joint>
             <actuator name="joint_${linkName}">
-                <hardwareInterface>hardware_interface/EffortJointInterface</hardwareInterface>
+                <hardwareInterface>hardware_interface/VelocityJointInterface</hardwareInterface>
                 <mechanicalReduction>1</mechanicalReduction>
             </actuator>
@@ -106,8 +106,8 @@
             <type>transmission_interface/SimpleTransmission</type>
             <joint name="joint_${linkName}">
-                <hardwareInterface>hardware_interface/EffortJointInterface</hardwareInterface>
+                <hardwareInterface>hardware_interface/VelocityJointInterface</hardwareInterface>
             </joint>
             <actuator name="motor_joint_${linkName}">
-                <hardwareInterface>hardware_interface/EffortJointInterface</hardwareInterface>
+                <hardwareInterface>hardware_interface/VelocityJointInterface</hardwareInterface>
                 <mechanicalReduction>1</mechanicalReduction>
             </actuator>

Commit message: cartographer 可以跑通了，但是建的图不正确，

File: urdf/car.xacro (robot description, xacro)
@@ -84,5 +84,32 @@
         <child link="hokuyo_link"/>
     </joint>
-    <!-- <link name="imu_link"/><joint name="base_to_imu" type="fixed"><axis rpy="0 0 0" xyz="0 0 0"/><parent link="base_link"/><child link="imu_link"/><origin rpy="0 0 0" xyz="0 0 .2"/></joint> -->
+    <link name="imu_link">
+        <!-- <inertial><origin xyz="0.0 0.0 -0.2" rpy="0.0 0.0 0.0"/><mass value="0.2"/><inertia ixx="0.0" ixy="0.0" ixz="0.0" iyy="0.0" iyz="0.0" izz="0.0"/></inertial><visual><origin xyz="0.0 0.0 0.0" rpy="0.0 0.0 0.0"/><geometry><box size="0.2 0.2 0.2"/></geometry><material ><color rgba="1.0 0.0 0.0 1.0"/></material></visual><collision><origin xyz="0.0 0.0 0.0" rpy="0.0 0.0 0.0"/><geometry><box size="0.2 0.2 0.2"/></geometry></collision> -->
+    </link>
+    <joint name="base_to_imu" type="fixed">
+        <parent link="base_footprint"/>
+        <child link="imu_link"/>
+        <!-- <origin xyz="0.25 0.8 1.2" rpy="0.0 0.0 0.0"/> -->
+        <origin xyz="0 0 0" rpy="0.0 0.0 0.0"/>
+    </joint>
+    <gazebo reference="imu_link">
+        <gravity>true</gravity>
+        <sensor name="imu_sensor" type="imu">
+            <always_on>true</always_on>
+            <update_rate>20</update_rate>
+            <visualize>true</visualize>
+            <topic>imu</topic>
+            <plugin filename="libgazebo_ros_imu_sensor.so" name="imu_plugin">
+                <topicName>imu</topicName>
+                <bodyName>imu_link</bodyName>
+                <updateRateHZ>10.0</updateRateHZ>
+                <gaussianNoise>0.0</gaussianNoise>
+                <xyzOffset>0 0 0</xyzOffset>
+                <rpyOffset>0 0 0</rpyOffset>
+                <frameName>imu_link</frameName>
+            </plugin>
+            <pose>0 0 0 0 0 0</pose>
+        </sensor>
+    </gazebo>
     <xacro:macro name="wheel" params="linkName xyz rpy">
         <joint name="base_to_${linkName}" type="continuous">
@@ -108,4 +135,14 @@
                     <cylinder length="0.2" radius="0.35"/>
                 </geometry>
+                <surface>
+                    <friction>
+                        <ode>
+                            <mu>0.5</mu>
+                            <mu2>0.5</mu2>
+                            <slip1>1.0</slip1>
+                            <slip2>1.0</slip2>
+                        </ode>
+                    </friction>
+                </surface>
             </collision>
             <inertial>
@@ -116,8 +153,5 @@
         </link>
         <gazebo reference="${linkName}">
-            <mu>10</mu>
-            <mu2>10</mu2>
-            <kp>100000000.0</kp>
-            <kd>10000.0</kd>
+            <!-- <mu1>0.9</mu1><mu2>0.9</mu2><kp>100000000.0</kp><kd>10000.0</kd> -->
         </gazebo>
         <!-- <transmission name="tran${linkName}"><type>transmission_interface/SimpleTransmission</type><joint name="base_to_${linkName}"><hardwareInterface>hardware_interface/EffortJointInterface</hardwareInterface></joint><actuator name="motor_${linkName}"><hardwareInterface>hardware_interface/EffortJointInterface</hardwareInterface><mechanicalReduction>1</mechanicalReduction></actuator></transmission> -->
